Commit message: my_robot_bringup package added

File: src/my_robot_description/urdf/common_properties.urdf.xacro (robot description, xacro)
@@ -7,3 +7,30 @@
         <color rgba="0.5 0.5 0.5 1"/>
     </material>
+    <xacro:macro name="box_inertia" params="m l w h xyz rpy">
+        <inertial>
+            <origin xyz="${xyz}" rpy="${rpy}"/>
+            <mass value="${m}"/>
+            <inertia ixx="${ (m/12)*(h*h + l*l)}" ixy="0" ixz="0"
+                     iyy="${(m/12)*(w*w + l*l)}" iyz="0"
+                     izz="${(m/12)*(w*w + h*h)}" />
+        </inertial>
+    </xacro:macro>
+    <xacro:macro name="cylinder_inertia" params="m r l xyz rpy">
+        <inertial>
+            <origin xyz="${xyz}" rpy="${rpy}"/>
+            <mass value="${m}"/>
+            <inertia ixx="${(m/12)*(3*r*r + l*l)}" ixy="0" ixz="0"
+                     iyy="${(m/12)*(3*r*r + l*l)}" iyz="0"
+                     izz="${(m/2)*r*r}"/>
+        </inertial>
+    </xacro:macro>
+    <xacro:macro name="sphere_inertia" params="m r xyz rpy">
+        <inertial>
+            <origin xyz="${xyz}" rpy="${rpy}"/>
+            <mass value="${m}"/>
+            <inertia ixx="${(2/5)*m*r*r}" ixy="0" ixz="0"
+                     iyy="${(2/5)*m*r*r}" iyz="0"
+                     izz="${(2/5)*m*r*r}"/>
+        </inertial>
+    </xacro:macro>
 </robot>

File: src/my_robot_description/urdf/mobile_base.urdf.xacro (robot description, xacro)
@@ -14,4 +14,12 @@
             <material name="blue"/>
         </visual>
+        <collision>
+            <geometry>
+                <box size="${base_length} ${base_width} ${base_height}"/>    <!--In meters(m)-->
+            </geometry>
+            <origin xyz="0 0 ${base_height/2.0}" rpy= "0 0 0"/>
+        </collision>
+        <xacro:box_inertia m="5.0" l="${2*base_length}" w="${2*base_width}" h="${2*base_height}"
+                            xyz="0 0 ${base_height/2.0}" rpy="0 0 0"/>
     </link>
     <xacro:macro name="wheel_link" params="prefix">
@@ -24,4 +32,12 @@
                 <material name="grey"/>
             </visual>
+            <collision>
+                <geometry>
+                    <cylinder radius="${wheel_radius}" length="${wheel_length}"/>
+                </geometry>
+                <origin xyz="0 0 0" rpy="${pi/2.0} 0 0"/>
+            </collision>
+            <xacro:cylinder_inertia m="1.0" r="${2*wheel_radius}" l="${2*wheel_length}"
+                                    xyz="0 0 0" rpy="${pi/2.0} 0 0"/>
         </link>
     </xacro:macro>
@@ -36,4 +52,12 @@
             <material name="grey"/>
         </visual>
+        <collision>
+            <geometry>
+                <sphere radius="${wheel_radius/2.0}"/>
+            </geometry>
+            <origin xyz="0 0 0" rpy="0 0 0"/>
+        </collision>
+        <xacro:sphere_inertia m="0.5" r="${2*wheel_radius/2.0}"
+                              xyz="0 0 0" rpy="0 0 0"/>
     </link>
     <link name="base_footprint">

File: src/my_robot_description/urdf/my_robot.urdf.xacro (robot description, xacro)
@@ -3,3 +3,4 @@
     <xacro:include filename="common_properties.urdf.xacro"/>
     <xacro:include filename="mobile_base.urdf.xacro"/>
+    <xacro:include filename="mobile_base_gazebo.xacro"/>
 </robot>

Commit message: Final Project Solution

File: src/my_robot_description/urdf/common_properties.urdf.xacro (robot description, xacro)
@@ -6,4 +6,10 @@
     <material name="grey">
         <color rgba="0.5 0.5 0.5 1"/>
+    </material>
+    <material name="orange">
+        <color rgba="1 0.62 0 1"/>
+    </material>
+    <material name="yellow">
+        <color rgba="1 0.98 0 1"/>
     </material>
     <xacro:macro name="box_inertia" params="m l w h xyz rpy">

File: src/my_robot_description/urdf/mobile_base_gazebo.xacro (robot description, xacro)
@@ -1,4 +1,5 @@
 <?xml version="1.0"?>
 <robot xmlns:xacro="http://www.ros.org/wiki/xacro">
+    <!--color compatibility with Gazebo and model plugin-->
     <gazebo reference="base_link">
         <material>Gazebo/Blue</material>

File: src/my_robot_description/urdf/my_robot.urdf.xacro (robot description, xacro)
@@ -4,3 +4,5 @@
     <xacro:include filename="mobile_base.urdf.xacro"/>
     <xacro:include filename="mobile_base_gazebo.xacro"/>
+    <xacro:include filename="camera.xacro"/>
+    <xacro:include filename="standalone_arm.urdf.xacro"/>
 </robot>
